File: PCB_Design/MiniBLDC/MOSFET.kicad_sch (KiCad schematic)
At the start: 9 parts, among them J6 Conn_02x02_Counter_Clockwise, Q1 BSC026N08NS5, Q2 BSC026N08NS5

Commit message: v2.0 done
Parts:
- J6: footprint Connector_PinHeader_2.54mm:PinHeader_2x02_P2.54mm_Vertical -> MountingHole:MountingHole_2.5mm_Pad_Via
Changed lines of the file:
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@@
       (effects (font (size 1.27 1.27)))
     )
-    (property "Footprint" "Connector_PinHeader_2.54mm:PinHeader_2x02_P2.54mm_Vertical" (at 236.22 83.82 0)
+    (property "Footprint" "MountingHole:MountingHole_2.5mm_Pad_Via" (at 236.22 83.82 0)
       (effects (font (size 1.27 1.27)) hide)
     )
