File: PCB_Design/MiniBLDC/MiniBLDC_v2_twoside_1_24_2024.kicad_pcb (KiCad board)
At the start: 4 copper layers, 46 x 46 mm, 123 parts, among them IC2 MAX17502EATB+T, IC3 WS2812B, J1 Conn_01x06_Pin, J13 Conn_01x02, J14 USB_C_Receptacle_USB2.0, J2 Conn_01x02, J3 Conn_01x02_Pin, J6 Conn_02x02_Counter_Clockwise, J7 Conn_02x02_Counter_Clockwise, J8 Conn_02x02_Counter_Clockwise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

Commit message: Move DC converter away from encoder
Parts:
- C22, C34, C35, C36: moved to F.Cu
- moved C22 14.2 mm to (148.1, 121.2), turned to -90 degrees
- moved C36 12.1 mm to (146.1, 117.6), turned to -90 degrees
- moved C21 11.7 mm to (151.6, 106.8)
- moved C33 11.7 mm to (148.3, 106.8)
- moved L1 11.6 mm to (149.9, 112.9)
- moved C35 11.3 mm to (144.7, 117.6), turned to -90 degrees
- moved C37 11.2 mm to (148.1, 122.3)
- moved C38 11.2 mm to (150.4, 122.3)
- moved IC2 11.1 mm to (148.8, 118.3)
- moved C34 10.9 mm to (143.2, 117.6), turned to -90 degrees
- moved C16 2.39 mm to (144.2, 118.7), turned to 180 degrees
- moved C17 2.37 mm to (144.2, 116.4), turned to 180 degrees
Routing:
- net MCU_D+: track 15.0 -> 25.0 mm
- net MCU_D-: track 13.4 -> 23.1 mm
- net GND: track 126.9 -> 117.5 mm, vias 133 -> 163
- net +3V3: track 72.6 -> 70.2 mm, vias 16 -> 18
- net /VM: track 64.8 -> 67.1 mm
- net Net-(IC2-VCC): track 4.18 -> 2.63 mm, vias 0 -> 1
- net Net-(IC2-SS): track 6.29 -> 4.82 mm, vias 2 -> 1
